File: src/kicad/capslock/capslock.kicad_pcb (KiCad board)
At the start: 2 copper layers, 25.4 x 12.1 mm, 12 parts, among them J1 USB_A, U1 PIC16(L)F1455-I/ST

Commit message: Gerbers used for ALLPCB job 2C036588
Other:
- board text removed: "Gold-plated fingers"
